File: concept2creation.kicad_pcb (KiCad board)
At the start: 2 copper layers, 44 x 58 mm, 29 parts, among them J1 XKB-USB-C16PIN, J2 CONN_061.27MM, J3 Conn_01x10, M1 HOLYIOT_18010, Q6 PMOSFETSOT23, U1 TP4054-42-SOT25-R_TP4054-42-S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, U2 XB3303ASOT23, U3 max8815aetb+, X1 BM02B-SRSS-TB

Commit message: concept2creation
Parts:
- moved LED1 17.0 mm to (50.0, 76.6)
- moved J1 7.47 mm to (30.0, 85.0)
- moved R99 7.25 mm to (33.6, 83.0), turned to 0 degrees
- moved S1 6.01 mm to (50.0, 70.6)
- moved R100 5.44 mm to (33.6, 86.2), turned to 0 degrees
- turned J3 to 180 degrees
Routing:
- net /RX: track 26.0 -> 99.8 mm
- net /TX: track 24.6 -> 97.7 mm
- net VBUS: track 117.8 -> 166.7 mm
- net D-: track 95.4 -> 137.0 mm
- net D+: track 94.8 -> 134.6 mm
- net +3.3V: track 40.7 -> 72.4 mm, vias 1 -> 2
- net +5V: track 39.4 -> 57.8 mm
- net GND: track 16.9 -> 27.2 mm, vias 14 -> 18
- net /NRF/RST: track 48.3 -> 56.2 mm
- net Net-(FUSE1-Pad1): track 14.3 -> 20.0 mm
- net /5VEN: track 32.9 -> 36.5 mm
- net V_RAW: track 29.2 -> 26.7 mm
- net /WS2812: track 20.5 -> 22.6 mm
- net /NRF/BVOLT: track 18.7 -> 19.5 mm
- net Net-(J1-CC2): track 2.26 -> 2.96 mm
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Other:
- board size 44 x 58 mm -> 48.2 x 80.1 mm
- board text added: "Sensor"
